File: LiPo-Charger MultiBoard/charger.sch (EAGLE design)
At the start: 25 parts, among them IC1 MCP73832T, IC2 MCP73832T

Commit message: Updated schematics and board. Added LibreOffice calculation for part lists.
Parts:
- FEMALE_B, FEMALE_R, MALE_L, MALE_T: device pinhead-2:PINHD-1X02_2.54-SMD-90° -> pinhead-2:PINHD-1X02_2.54-90°
- FEMALE_BL, FEMALE_BR, FEMALE_RB, FEMALE_RT, MALE_LB, MALE_LT, MALE_TL, MALE_TR: device pinhead-2:PINHD-1X04_2.54-SMD-90° -> pinhead-2:PINHD-1X04_2.54-90°
- R1, R3: value 130R -> 470R
- R2, R4: value 2k -> 5k6
Connections:
- net +5V: now also R1.2, R3.2; no longer R1.1, R3.1
- net N$2: now also R1.1; no longer R1.2
- net N$5: now also R3.1; no longer R3.2
Other:
- moved on the sheet: R1, R3
Changed lines of the file:
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@@
 <setting verticaltext="up"/>
 </settings>
-<grid distance="0.1" unitdist="inch" unit="inch" style="lines" multiple="1" display="yes" altdistance="0.01" altunitdist="inch" altunit="inch"/>
+<grid distance="0.1" unitdist="inch" unit="inch" style="lines" multiple="1" display="no" altdistance="0.01" altunitdist="inch" altunit="inch"/>
 <layers>
 <layer number="1" name="Top" color="4" fill="1" visible="no" active="no"/>
@@
 <parts>
 <part name="IC1" library="microchip" deviceset="MCP73832T-2DCI/OT" device="" value="MCP73832T"/>
-<part name="R1" library="rcl" deviceset="R-EU_" device="R1206" value="130R"/>
-<part name="R2" library="rcl" deviceset="R-EU_" device="R1206" value="2k"/>
+<part name="R1" library="rcl" deviceset="R-EU_" device="R1206" value="470R"/>
+<part name="R2" library="rcl" deviceset="R-EU_" device="R1206" value="5k6"/>
 <part name="C1" library="rcl" deviceset="C-EU" device="C1206" value="4.7µ, 5V"/>
 <part name="LED1" library="led" deviceset="LED" device="CHIPLED_1206" value="red"/>
@@
 <part name="GND4" library="supply1" deviceset="GND" device=""/>
 <part name="IC2" library="microchip" deviceset="MCP73832T-2DCI/OT" device="" value="MCP73832T"/>
-<part name="R3" library="rcl" deviceset="R-EU_" device="R1206" value="130R"/>
-<part name="R4" library="rcl" deviceset="R-EU_" device="R1206" value="2k"/>
+<part name="R3" library="rcl" deviceset="R-EU_" device="R1206" value="470R"/>
+<part name="R4" library="rcl" deviceset="R-EU_" device="R1206" value="5k6"/>
 <part name="C2" library="rcl" deviceset="C-EU" device="C1206" value="4.7µ, 5V"/>
 <part name="LED2" library="led" deviceset="LED" device="CHIPLED_1206" value="red"/>
@@
 <part name="GND6" library="supply1" deviceset="GND" device=""/>
 <part name="FRAME1" library="frames" deviceset="A4L-LOC" device=""/>
-<part name="MALE_TL" library="pinhead-2" deviceset="PINHD-1X04" device="_2.54-SMD-90°"/>
-<part name="MALE_TR" library="pinhead-2" deviceset="PINHD-1X04" device="_2.54-SMD-90°"/>
-<part name="MALE_LT" library="pinhead-2" deviceset="PINHD-1X04" device="_2.54-SMD-90°"/>
-<part name="MALE_LB" library="pinhead-2" deviceset="PINHD-1X04" device="_2.54-SMD-90°"/>
+<part name="MALE_TL" library="pinhead-2" deviceset="PINHD-1X04" device="_2.54-90°"/>
+<part name="MALE_TR" library="pinhead-2" deviceset="PINHD-1X04" device="_2.54-90°"/>
+<part name="MALE_LT" library="pinhead-2" deviceset="PINHD-1X04" device="_2.54-90°"/>
+<part name="MALE_LB" library="pinhead-2" deviceset="PINHD-1X04" device="_2.54-90°"/>
 <part name="P+5" library="supply1" deviceset="+5V" device=""/>
 <part name="GND7" library="supply1" deviceset="GND" device=""/>
 <part name="+3V2" library="supply1" deviceset="+3V3" device=""/>
-<part name="FEMALE_RT" library="pinhead-2" deviceset="PINHD-1X04" device="_2.54-SMD-90°"/>
-<part name="FEMALE_RB" library="pinhead-2" deviceset="PINHD-1X04" device="_2.54-SMD-90°"/>
-<part name="FEMALE_BL" library="pinhead-2" deviceset="PINHD-1X04" device="_2.54-SMD-90°"/>
-<part name="FEMALE_BR" library="pinhead-2" deviceset="PINHD-1X04" device="_2.54-SMD-90°"/>
+<part name="FEMALE_RT" library="pinhead-2" deviceset="PINHD-1X04" device="_2.54-90°"/>
+<part name="FEMALE_RB" library="pinhead-2" deviceset="PINHD-1X04" device="_2.54-90°"/>
+<part name="FEMALE_BL" library="pinhead-2" deviceset="PINHD-1X04" device="_2.54-90°"/>
+<part name="FEMALE_BR" library="pinhead-2" deviceset="PINHD-1X04" device="_2.54-90°"/>
 <part name="P+6" library="supply1" deviceset="+5V" device=""/>
 <part name="GND8" library="supply1" deviceset="GND" device=""/>
-<part name="MALE_T" library="pinhead-2" deviceset="PINHD-1X02" device="_2.54-SMD-90°"/>
-<part name="MALE_L" library="pinhead-2" deviceset="PINHD-1X02" device="_2.54-SMD-90°"/>
-<part name="FEMALE_R" library="pinhead-2" deviceset="PINHD-1X02" device="_2.54-SMD-90°"/>
-<part name="FEMALE_B" library="pinhead-2" deviceset="PINHD-1X02" device="_2.54-SMD-90°"/>
+<part name="MALE_T" library="pinhead-2" deviceset="PINHD-1X02" device="_2.54-90°"/>
+<part name="MALE_L" library="pinhead-2" deviceset="PINHD-1X02" device="_2.54-90°"/>
+<part name="FEMALE_R" library="pinhead-2" deviceset="PINHD-1X02" device="_2.54-90°"/>
+<part name="FEMALE_B" library="pinhead-2" deviceset="PINHD-1X02" device="_2.54-90°"/>
 <part name="BOT_CON" library="con-hirose" deviceset="DF12-20" device="DS"/>
 <part name="+3V3" library="supply1" deviceset="+3V3" device=""/>
@@
 <instances>
 <instance part="IC1" gate="A" x="109.22" y="152.4"/>
-<instance part="R1" gate="G$1" x="78.74" y="160.02" rot="R270"/>
+<instance part="R1" gate="G$1" x="78.74" y="160.02" rot="R90"/>
 <instance part="R2" gate="G$1" x="129.54" y="139.7" rot="R90"/>
 <instance part="C1" gate="G$1" x="88.9" y="139.7"/>
@@
 <instance part="GND4" gate="1" x="88.9" y="129.54"/>
 <instance part="IC2" gate="A" x="109.22" y="99.06"/>
-<instance part="R3" gate="G$1" x="78.74" y="106.68" rot="R270"/>
+<instance part="R3" gate="G$1" x="78.74" y="106.68" rot="R90"/>
 <instance part="R4" gate="G$1" x="129.54" y="86.36" rot="R90"/>
 <instance part="C2" gate="G$1" x="88.9" y="86.36"/>
@@
 <segment>
 <pinref part="LED1" gate="G$1" pin="A"/>
-<pinref part="R1" gate="G$1" pin="2"/>
 <wire x1="81.28" y1="152.4" x2="78.74" y2="152.4" width="0.1524" layer="91"/>
+<pinref part="R1" gate="G$1" pin="1"/>
 <wire x1="78.74" y1="152.4" x2="78.74" y2="154.94" width="0.1524" layer="91"/>
 </segment>
 </net>
 <net name="+5V" class="0">
-<segment>
-<pinref part="R1" gate="G$1" pin="1"/>
-<wire x1="78.74" y1="165.1" x2="78.74" y2="167.64" width="0.1524" layer="91"/>
-<pinref part="P+1" gate="1" pin="+5V"/>
-</segment>
 <segment>
 <pinref part="IC1" gate="A" pin="VDD"/>
@@
 <wire x1="127" y1="149.86" x2="132.08" y2="149.86" width="0.1524" layer="91"/>
 <wire x1="132.08" y1="149.86" x2="132.08" y2="167.64" width="0.1524" layer="91"/>
-</segment>
-<segment>
-<pinref part="R3" gate="G$1" pin="1"/>
-<wire x1="78.74" y1="111.76" x2="78.74" y2="114.3" width="0.1524" layer="91"/>
-<pinref part="P+3" gate="1" pin="+5V"/>
 </segment>
 <segment>
@@
 <wire x1="160.02" y1="116.84" x2="160.02" y2="124.46" width="0.1524" layer="91"/>
 <junction x="160.02" y="116.84"/>
+</segment>
+<segment>
+<pinref part="R1" gate="G$1" pin="2"/>
+<pinref part="P+1" gate="1" pin="+5V"/>
+<wire x1="78.74" y1="165.1" x2="78.74" y2="167.64" width="0.1524" layer="91"/>
+</segment>
+<segment>
+<pinref part="R3" gate="G$1" pin="2"/>
+<pinref part="P+3" gate="1" pin="+5V"/>
+<wire x1="78.74" y1="111.76" x2="78.74" y2="114.3" width="0.1524" layer="91"/>
 </segment>
 </net>
@@
 <segment>
 <pinref part="LED2" gate="G$1" pin="A"/>
-<pinref part="R3" gate="G$1" pin="2"/>
 <wire x1="81.28" y1="99.06" x2="78.74" y2="99.06" width="0.1524" layer="91"/>
+<pinref part="R3" gate="G$1" pin="1"/>
 <wire x1="78.74" y1="99.06" x2="78.74" y2="101.6" width="0.1524" layer="91"/>
 </segment>
