File: LiPo-Charger-Station/lipo-charger-station.brd (EAGLE design)
At the start: 201.9 x 130.6 mm, 126 parts, among them IC1 AP1084D33G-13, IC100 ATMEGA8A-AU, IC2 LT1083CP-5, T1 EVQQ2F03W, T2 EVQQ2F03W, T3 EVQQ2F03W, T4 EVQQ2F03W, U1 MCP73831T-2ATI/OT, U10 MCP73831T-2ATI/OT, U11 MCP73831T-2ATI/OT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

Commit message: Fixed errors in LiPo-Charger-Station
Parts:
- moved IC1 10.4 mm to (130.8, 109.2), turned to 90 degrees
Connections:
- net +12V: now also IC1.2; no longer IC1.3
- net +3V3: now also IC1.3; no longer IC1.2
Routing:
- net +3V3: track 543.8 -> 553.3 mm
- net +5V: track 1030.4 -> 1034.5 mm, vias 20 -> 21
- net +12V: track 64.3 -> 67.0 mm
- added copper zone on layer 1, net N$27
Other:
- board text added: "GND"
- board text added: "VCC"
