File: mrShark/mrShark 1.2/mrShark 12.sch (EAGLE design)
At the start: 78 parts, among them IC1 ATMEGA168-20MU, IC2 PCA9540BDP, IC3 TIR1000PWR, IC4 TFBS4711TR1, IC5 DRV8830DRCT, IC6 LTC2990IMS#PBF, IC7 DRV8830DRCT, IC8 LTC2990IMS#PBF, Q1 TXC - 7X-1.8432MBB-T - OSC, 1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, Q2 BC817W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

Commit message: Updated mrShark 1.2 & 1.3 Updated mrShark Adapter Updated mrShark LED-Marker to version 0.0.3
Connections:
- net BAT1: now also IC8.V1
- net BAT1+: no longer IC8.V1
- net BAT2: now also IC8.V2
- net BAT2+: no longer IC8.V2
Changed lines of the file:
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@@
 <?xml version="1.0" encoding="utf-8"?>
 <!DOCTYPE eagle SYSTEM "eagle.dtd">
-<eagle version="7.1.0">
+<eagle version="6.3">
 <drawing>
 <settings>
@@
 <setting verticaltext="up"/>
 </settings>
-<grid distance="0.1" unitdist="inch" unit="inch" style="lines" multiple="1" display="no" altdistance="0.01" altunitdist="inch" altunit="inch"/>
+<grid distance="0.1" unitdist="inch" unit="inch" style="lines" multiple="1" display="yes" altdistance="0.01" altunitdist="inch" altunit="inch"/>
 <layers>
 <layer number="1" name="Top" color="4" fill="1" visible="no" active="no"/>
@@
 <net name="BAT1+" class="0">
 <segment>
-<pinref part="IC8" gate="A" pin="V1"/>
-<wire x1="121.92" y1="53.34" x2="111.76" y2="53.34" width="0.1524" layer="91"/>
-<label x="111.76" y="53.34" size="1.27" layer="95" rot="R180" xref="yes"/>
-</segment>
-<segment>
 <pinref part="SWITCH_PWR" gate="T1" pin="O"/>
 <pinref part="D1" gate="G$1" pin="A"/>
 <wire x1="81.28" y1="144.78" x2="83.82" y2="144.78" width="0.1524" layer="91"/>
+<label x="83.82" y="144.78" size="1.27" layer="95" rot="R90"/>
 </segment>
 </net>
 <net name="BAT2+" class="0">
-<segment>
-<pinref part="IC8" gate="A" pin="V2"/>
-<wire x1="121.92" y1="50.8" x2="111.76" y2="50.8" width="0.1524" layer="91"/>
-<label x="111.76" y="50.8" size="1.27" layer="95" rot="R180" xref="yes"/>
-</segment>
 <segment>
 <pinref part="SWITCH_PWR" gate="T1" pin="O1"/>
 <pinref part="D2" gate="G$1" pin="A"/>
 <wire x1="81.28" y1="134.62" x2="83.82" y2="134.62" width="0.1524" layer="91"/>
+<label x="83.82" y="134.62" size="1.27" layer="95" rot="R90"/>
 </segment>
 </net>
@@
 <label x="48.26" y="149.86" size="1.27" layer="95"/>
 </segment>
+<segment>
+<pinref part="IC8" gate="A" pin="V1"/>
+<wire x1="121.92" y1="53.34" x2="111.76" y2="53.34" width="0.1524" layer="91"/>
+<label x="111.76" y="53.34" size="1.27" layer="95" rot="R180" xref="yes"/>
+</segment>
 </net>
 <net name="BAT2" class="0">
@@
 <label x="48.26" y="124.46" size="1.27" layer="95"/>
 </segment>
-</net>
+<segment>
+<pinref part="IC8" gate="A" pin="V2"/>
+<wire x1="121.92" y1="50.8" x2="111.76" y2="50.8" width="0.1524" layer="91"/>
+<label x="111.76" y="50.8" size="1.27" layer="95" rot="R180" xref="yes"/>
+</segment>
+</net>
