File: mrShark/mrShark 1.3/mrShark 13.sch (EAGLE design)
At the start: 78 parts, among them IC1 ATMEGA168-20MU, IC2 PCA9540BDP, IC3 TIR1000PWR, IC4 TFBS4711TR1, IC5 DRV8830DRCT, IC6 LTC2990IMS#PBF, IC7 DRV8830DRCT, IC8 LTC2990IMS#PBF, Q1 TXC - 7X-1.8432MBB-T - OSC, 1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, Q2 BC817W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

Commit message: Updated mrShark 1.2 & 1.3 Updated mrShark Adapter Updated mrShark LED-Marker to version 0.0.3
Parts:
- R6: value 100R -> 87R
Changed lines of the file:
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@@
 <setting verticaltext="up"/>
 </settings>
-<grid distance="0.1" unitdist="inch" unit="inch" style="lines" multiple="1" display="yes" altdistance="0.01" altunitdist="inch" altunit="inch"/>
+<grid distance="0.1" unitdist="inch" unit="inch" style="lines" multiple="1" display="no" altdistance="0.01" altunitdist="inch" altunit="inch"/>
 <layers>
 <layer number="1" name="Top" color="4" fill="1" visible="no" active="no"/>
@@
 <part name="R33" library="rcl" deviceset="R-EU_" device="R0201" value="200R"/>
 <part name="GND9" library="supply1" deviceset="GND" device=""/>
-<part name="R6" library="rcl" deviceset="R-EU_" device="R0201" value="100R"/>
+<part name="R6" library="rcl" deviceset="R-EU_" device="R0201" value="87R"/>
 <part name="LED1" library="led" deviceset="LED" device="CHIPLED_0603" value="green"/>
 <part name="GND10" library="supply1" deviceset="GND" device=""/>
