File: mrShark/mrShark 0.6/v1/ultrasonic v1.sch (EAGLE design)
At the start: 78 parts, among them IC1 ATMEGA168-20MU, IC2 PCA9540BDP, IC3 TIR1000PWR, IC4 TFBS4711TR1, IC5 DRV8830DRCT, IC6 LTC2990IMS#PBF, IC7 DRV8830DRCT, IC8 LTC2990IMS#PBF, Q1 TXC - 7X-1.8432MBB-T - OSC, 1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, Q2 BC817W, Q3 BC817W, Q4 BC817W, Q5 BC817W, Q6 BC817W, Q7 BC817W, Q8 BC817W, Q9 14,7456MHZ

Commit message: Updated Board layouts an schematics
Parts:
- removed BAT1+1, BAT1-1, BAT2+1, BAT2-1, MOT1, MOT2, MOT3, MOT4: (no value), wirepad:1,6/0,9
- removed C2: 100n, rcl:C-EUC0201
- removed C3, C4: 18p, rcl:C-EUC0201
- removed C5: 10µ, rcl:C-EUC0603K
- removed CON_PROG: DF12(5.0)-20DP-0.5V, con-hirose:DF12-20DP
- removed D1, D2: PMEG2010EA, diode:PMEG2010EAR
- removed H1, H2, H3, H4: MOUNT-HOLE1,5, holes:MOUNT-HOLE1,5
- removed IC2: PCA9540BDP, nxp:PCA9540TSSOP8
- removed IC3: TIR1000PWR, texas:TIR1000PWR
- removed IC4: TFBS4711TR1, vishay:TFBS4711TR1
- removed IC5, IC7: DRV8830DRCT, texas:DRV8830DGQRWSON
- removed IC6, IC8: LTC2990IMS#PBF, linear-technology:LTC2990IMSPBF
- removed LED4, LED5: ASMT-YTD2-0BB02, led:PLCC6K
- removed LED6: red, led:LEDCHIPLED_0603
- removed Q1: TXC - 7X-1.8432MBB-T - OSC, 1.8432MHZ, crystal:7X-SERIES
- removed Q2, Q3, Q4, Q5, Q6, Q7, Q8: BC817W, transistor-npn:BC817W
- removed Q9: 14,7456MHZ, crystal:TXC-7B-SERIESSMD
- removed R10: 27R, rcl:R-EU_R0201
- removed R11, R13: 2k, rcl:R-EU_R0201
- removed R12: 1k, rcl:R-EU_R0201
- removed R14, R15, R16, R17, R18, R23, R24, R9: 100k, rcl:R-EU_R0201
- removed R19, R20, R25, R26: 560R, rcl:R-EU_R0201
- removed R21, R22, R27, R28: 130R, rcl:R-EU_R0201
- removed R29, R31: 0.91R, rcl:R-EU_R0603
- removed R30, R32: 0R2, rcl:R-EU_R0603
- removed R33: 39R, rcl:R-EU_R0603
- removed R34, R35: 1k8, rcl:R-EU_R0402
- removed R7, R8: 1k8, rcl:R-EU_R0201
- removed SWITCH_PWR: AYZ0202AGRLC, switch:AYZ0202AGRLC
- added ISP: (no value), con-ml:ML10L
- added R3: 68R, rcl:R-EU_R0805W
- added SERVO1, SERVO2, SERVO3, SERVO4, SERVO5, SERVO6: (no value), pinhead:PINHD-1X3
- added U$1: (no value), Tim:ADAPTER_BLANKO_3X5B2
- added US1, US2, US3, US4, US5, US6: (no value), pinhead:PINHD-1X4
- C1: device rcl:C-EUC0201 -> rcl:C-EUC0805
- IC1: value ATMEGA168-20MU -> ATtiny48; device atmega8:ATMEGA48/88/168-MU -> atmega8:ATMEGA8-AU
- LED1: device led:LEDCHIPLED_0603 -> led:LEDCHIP-LED0805
- LED2, LED3: value ASMT-YTD2-0BB02 -> rot; device led:PLCC6K -> led:LEDCHIP-LED0805
- R1: value 100k -> 1k; device rcl:R-EU_R0201 -> rcl:R-EU_R0805W
- R2, R5: value 100k -> 1k8; device rcl:R-EU_R0201 -> rcl:R-EU_R0805W
- R4: value 100k -> 150R; device rcl:R-EU_R0201 -> rcl:R-EU_R0805W
- R6: value 82R -> 150R; device rcl:R-EU_R0603 -> rcl:R-EU_R0805W
Connections:
- removed net ADC7: CON_PROG.17, IC1.ADC7
- removed net BAT1: BAT1+1.P, SWITCH_PWR.P
- removed net BAT1+: D1.A, IC8.V1, SWITCH_PWR.O
- removed net BAT2: BAT2+1.P, SWITCH_PWR.P1
- removed net BAT2+: D2.A, IC8.V2, SWITCH_PWR.O1
- removed net CLK: IC3.CLK, Q1.FO
- removed net COLOR_B: LED2.BC, LED3.BC, LED4.BC, LED5.BC, Q4.C
- removed net COLOR_G: LED2.GC, LED3.GC, LED4.GC, LED5.GC, Q2.C
- removed net COLOR_R: LED2.RC, LED3.RC, LED4.RC, LED5.RC, Q3.C
- removed net I2C_ADC0: CON_PROG.13, IC8.V3
- removed net I2C_ADC1: CON_PROG.12, IC8.V4
- removed net INT0: CON_PROG.4, IC1.PD2(INT0/PCINT18), R4.2
- removed net INT1: CON_PROG.3, IC1.PD3(INT1/OC2B/PCINT19), R5.2
- removed net IRDA: IC4.IRDA, R10.2
- removed net IR_SD: IC1.PD4(T0/XCK/PCINT20), IC4.SD, R9.1
- removed net LED1: IC1.PD6(AIN0/OC0A/PCINT22), R17.2, R19.1
- removed net LED2: IC1.PC3(ADC3/PCINT11), R18.2, R20.1
- removed net LED3: IC1.PD5(T1/OC0B/PCINT21), R23.2, R25.1
- removed net LED4: IC1.PC2(ADC2/PCINT10), R24.2, R26.1
- removed net LED_B: IC1.PB1(OC1A/PCINT1), R13.2
- removed net LED_G: IC1.PB0(ICP1/CLKO/PCINT0), R11.2
- removed net LED_R: IC1.PD7(AIN1/PCINT23), R12.2
- removed net N$10: LED4.RA, R27.1
- removed net N$11: LED4.BA, LED4.GA, Q7.E, R27.2
- removed net N$15: LED3.RA, R22.1
- removed net N$16: LED3.BA, LED3.GA, Q6.E, R22.2
- removed net N$19: Q6.B, R20.2
- removed net N$20: LED5.RA, R28.1
- removed net N$22: LED5.BA, LED5.GA, Q8.E, R28.2
- removed net N$23: Q8.B, R26.2
- removed net N$24: Q7.B, R25.2
- removed net N$25: Q5.B, R19.2
- removed net N$26: C2.1, IC1.AREF
- removed net N$27: LED2.BA, LED2.GA, Q5.E, R21.2
- removed net N$28: LED6.A, R33.1
- removed net N$3: IC1.PB2(SS/OC1B/PCINT2), R6.1
- removed net N$4: Q1.OE, R1.2
- removed net N$5: LED2.RA, R21.1
- removed net N$8: LED1.A, R6.2
- removed net P_BAT1+: CON_PROG.14, SWITCH_PWR.S
- removed net P_BAT2+: CON_PROG.15, SWITCH_PWR.S1
- removed net RI2C_EN: IC1.ADC6
- removed net RSCL: CON_PROG.8, IC1.PC5(ADC5/SCL/PCINT13), IC2.SCL, R34.1
- removed net RSDA: CON_PROG.9, IC1.PC4(ADC4/SDA/PCINT12), IC2.SDA, R35.1
- removed net RXD: IC1.PD0(RXD/PCINT16), IC3.RXD
- removed net RXIR: IC3.IR_RXD, IC4.RXD
- removed net SENS_MOTL1: IC5.OUT1, IC6.V1, R30.1
- removed net SENS_MOTL2: IC6.V2, MOT2.P, R30.2
- removed net SENS_MOTR1: IC6.V3, IC7.OUT1, R32.1
- removed net SENS_MOTR2: IC6.V4, MOT4.P, R32.2
- removed net SRXD: CON_PROG.11, IC1.PC0(ADC0/PCINT8)
- removed net STXD: CON_PROG.10, IC1.PC1(ADC1/PCINT9)
- removed net TXD: IC1.PD1(TXD/PCINT17), IC3.TXD
- removed net TXIR: IC3.IR_TXD, IC4.TXD
- removed net VCC: C1.1, C5.1, CON_PROG.1, D1.C, D2.C, IC1.AVCC, IC1.VCC@1, IC1.VCC@2, IC2.VCC, IC3.VCC, IC4.VCC, IC5.VCC, IC6.VCC, IC7.A0, IC7.VCC, IC8.ADR0, IC8.VCC, Q1.VCC, Q5.C, Q6.C, Q7.C, Q8.C, R1.1, R10.1, R2.1, R33.2, R34.2, R35.2, R4.1, R5.1, R7.2, R8.2
- removed net X1: Q4.B, R13.1, R16.2
- removed net X2: Q3.B, R12.1, R15.2
- removed net X3: Q2.B, R11.1, R14.2
- removed net XTAL1: C3.1, IC1.PB6(XTAL1/TOSC1/PCINT6), Q9.2
- removed net XTAL2: C4.1, IC1.PB7(XTAL2/TOSC2/PCINT7), Q9.1
- new net +5V: IC1.VCC@1, IC1.VCC@2, ISP.2, R1.1, R2.1, R4.2, R5.1, SERVO1.2, SERVO2.2, SERVO3.2, SERVO4.2, SERVO5.2, SERVO6.2, U$1.5V, US1.1, US2.1, US3.1, US4.1, US5.1, US6.1
- new net N$9: C1.1, IC1.AREF
- new net SERVO1: IC1.PD0(RXD), SERVO1.1
- new net SERVO2: IC1.PD1(TXD), SERVO2.1
- new net SERVO3: IC1.PD2(INT0), SERVO3.1
- new net SERVO4: IC1.PD3(INT1), SERVO4.1
- new net SERVO5: IC1.PD4(T0/XCK), SERVO5.1
- new net SERVO6: IC1.PD5(T1), SERVO6.1
- new net US1_ECHO: IC1.ADC6, US1.3
- new net US1_TRIG: IC1.PD6(AIN0), US1.2
- new net US2_ECHO: IC1.ADC7, US2.3
- new net US2_TRIG: IC1.PB6(XTAL1/TOSC1), US2.2
- new net US3_ECHO: IC1.PC0(ADC0), US3.3
- new net US3_TRIG: IC1.PD7(AIN1), US3.2
- new net US4_ECHO: IC1.PC1(ADC1), US4.3
- new net US4_TRIG: IC1.PB0(ICP1), US4.2
- new net US5_ECHO: IC1.PC2(ADC2), US5.3
- new net US5_TRIG: IC1.PB1(OC1A), US5.2
- new net US6_ECHO: IC1.PC3(ADC3), US6.3
- new net US6_TRIG: IC1.PB2(SS/OC1B), US6.2
- net GND: now also ISP.10, ISP.4, ISP.6, ISP.8, LED2.C, LED3.C, SERVO1.3, SERVO2.3, SERVO3.3, SERVO4.3, SERVO5.3, SERVO6.3, U$1.GND, US1.4, US2.4, US3.4, US4.4, US5.4, US6.4; no longer BAT1-1.P, BAT2-1.P, C2.2, C3.2, C4.2, C5.2, CON_PROG.16, CON_PROG.2, CON_PROG.5, IC2.GND, IC3.GND, IC3.RESET, IC4.GND, IC5.A0, IC5.A1, IC5.EP, IC5.GND, IC6.ADR0, IC6.ADR1, IC6.GND, IC7.A1, IC7.EP, IC7.GND, IC8.ADR1, IC8.GND, LED6.C, Q1.GND, Q2.E, Q3.E, Q4.E, R14.1, R15.1, R16.1, R17.1, R18.1, R23.1, R24.1, R29.1, R31.1, R9.2
- net MISO: now also IC1.PB4(MISO), ISP.9; no longer CON_PROG.19, IC1.PB4(MISO/PCINT4)
- net MOSI: now also IC1.PB3(MOSI/OC2), ISP.1; no longer CON_PROG.20, IC1.PB3(MOSI/OC2A/PCINT3)
- net N$1: now also IC1.PB7(XTAL2/TOSC2), R6.2; no longer IC5.OUT2, MOT1.P
- net N$2: now also LED3.A, R6.1; no longer IC5.ISENSE, R29.2
- net N$6: now also LED1.A, R3.2; no longer IC7.OUT2, MOT3.P
- net N$7: now also LED2.A, R4.1; no longer IC7.ISENSE, R31.2
- net RESET: now also IC1.PC6(/RESET), ISP.5, R1.2; no longer CON_PROG.7, IC1.PC6(/RESET/PCINT14), R2.2
- net SCK: now also IC1.PB5(SCK), ISP.7, R3.1; no longer CON_PROG.18, IC1.PB5(SCK/PCINT5)
- net SCL: now also IC1.PC5(ADC5/SCL), R5.2, U$1.SCL; no longer IC2.SC0, IC5.SCL, IC6.SCL, IC7.SCL, IC8.SCL, R8.1
- net SDA: now also IC1.PC4(ADC4/SDA), R2.2, U$1.SDA; no longer IC2.SD0, IC5.SDA, IC6.SDA, IC7.SDA, IC8.SDA, R7.1
Other:
- note added: "6x US-Sensor & Servo"
- note added: "Fachhochschule Kiel Robotik Labor Grenzstraße 5 24149 Kiel"
- note removed: "24149 Kiel"
- note removed: "CONNECTORS"
- note removed: "Controller / IR"
- note removed: "Fachbereich IuE"
- note removed: "Fachhochschule Kiel"
- note removed: "Grenzstraße 5"
- note removed: "LEDs"
- note removed: "MCCA000517"
- note removed: "MOTORS"
- note removed: "NorthernStars"
- note removed: "www.northern-stars.de"
