File: mrShark/mrShark Adapter/mrShark Adapter.brd (EAGLE design)
At the start: 26 x 31 mm, 23 parts, among them CON1 DF12-20DS, IC1 LM317MBSTT3, IC2 MCP73832T-2DCI/OT, IC3 MCP73832T-2DCI/OT, IC4 FT232RQ

Commit message: Updated to new connector layout.
Routing:
- net MISO: track 20.8 -> 19.9 mm
- net SCK: track 19.7 -> 20.5 mm
Other:
- board text added: "FH Kiel mrShark Adapter v0.0.1a"
- board text removed: "NorthernStars mrShark Adapter v0.0.1a"
Changed lines of the file:
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@@
 <?xml version="1.0" encoding="utf-8"?>
 <!DOCTYPE eagle SYSTEM "eagle.dtd">
-<eagle version="6.3">
+<eagle version="7.2.0">
 <drawing>
 <settings>
@@
 <setting verticaltext="up"/>
 </settings>
-<grid distance="19.685039" unitdist="mil" unit="mil" style="lines" multiple="1" display="yes" altdistance="0.025" altunitdist="inch" altunit="inch"/>
+<grid distance="10" unitdist="mil" unit="mil" style="lines" multiple="1" display="yes" altdistance="0.025" altunitdist="inch" altunit="inch"/>
 <layers>
 <layer number="1" name="Top" color="4" fill="1" visible="yes" active="yes"/>
@@
 <wire x1="14.5" y1="3" x2="21" y2="3" width="0" layer="20"/>
 <wire x1="21" y1="3" x2="21" y2="-0.5" width="0" layer="20"/>
-<text x="8.5" y="21" size="0.6096" layer="25">NorthernStars
+<text x="8.5" y="21" size="0.6096" layer="25" font="vector" ratio="15">FH Kiel
 mrShark Adapter
 v0.0.1a</text>
@@
 <pass name="Default">
 <param name="RoutingGrid" value="50mil"/>
+<param name="AutoGrid" value="1"/>
+<param name="Efforts" value="0"/>
+<param name="TopRouterVariant" value="1"/>
 <param name="tpViaShape" value="round"/>
 <param name="PrefDir.1" value="|"/>
@@
 </element>
 <element name="C1" library="rcl" package="C0603" value="100n" x="10" y="11" smashed="yes" rot="R180">
-<attribute name="NAME" x="9.365" y="12.135" size="0.6096" layer="25"/>
+<attribute name="NAME" x="9.365" y="11.881" size="0.6096" layer="25"/>
 <attribute name="VALUE" x="10.635" y="12.905" size="1.27" layer="27" rot="R180"/>
 </element>
@@
 </element>
 <element name="D2" library="diode" package="SOD323-R" value="PMEG2010EA" x="12.5" y="13.5" smashed="yes" rot="R90">
-<attribute name="NAME" x="11.5" y="12.4" size="0.6096" layer="25" rot="R90"/>
+<attribute name="NAME" x="11.5" y="12.654" size="0.6096" layer="25" rot="R90"/>
 <attribute name="VALUE" x="14.8" y="12.4" size="1.27" layer="27" rot="R90"/>
 </element>
@@
 <wire x1="9.25" y1="14.25" x2="9" y2="14" width="0.3048" layer="16"/>
 <wire x1="9" y1="14" x2="9" y2="12" width="0.3048" layer="16"/>
-<wire x1="9" y1="12" x2="9.5" y2="11.5" width="0.3048" layer="16"/>
-<wire x1="9.5" y1="11.5" x2="13.5" y2="11.5" width="0.3048" layer="16"/>
-<wire x1="13.5" y1="11.5" x2="14" y2="11" width="0.3048" layer="16"/>
-<via x="14" y="11" extent="1-16" drill="0.3048" shape="octagon"/>
-<wire x1="14" y1="11" x2="14.5" y2="10.5" width="0.3048" layer="1"/>
+<via x="14" y="9.746" extent="1-16" drill="0.3048" shape="octagon"/>
 <wire x1="14.5" y1="10.5" x2="21" y2="10.5" width="0.3048" layer="1"/>
 <wire x1="21" y1="10.5" x2="22" y2="9.5" width="0.3048" layer="1"/>
 <wire x1="22" y1="9.5" x2="23.08" y2="9.5" width="0.3048" layer="1"/>
 <wire x1="23.08" y1="9.5" x2="23.31" y2="9.27" width="0.3048" layer="1"/>
+<wire x1="9" y1="12" x2="11.254" y2="9.746" width="0.3048" layer="16"/>
+<wire x1="14" y1="9.746" x2="11.254" y2="9.746" width="0.3048" layer="16"/>
+<wire x1="14" y1="9.746" x2="14" y2="10" width="0.3048" layer="1"/>
+<wire x1="14" y1="10" x2="14.5" y2="10.5" width="0.3048" layer="1"/>
 </signal>
 <signal name="MISO">
@@
 <wire x1="9.75" y1="13.75" x2="9.5" y2="13.5" width="0.3048" layer="16"/>
 <wire x1="9.5" y1="13.5" x2="9.5" y2="12.5" width="0.3048" layer="16"/>
-<wire x1="9.5" y1="12.5" x2="10" y2="12" width="0.3048" layer="16"/>
-<wire x1="10" y1="12" x2="14.5" y2="12" width="0.3048" layer="16"/>
-<wire x1="14.5" y1="12" x2="15" y2="11.5" width="0.3048" layer="16"/>
-<wire x1="15" y1="11.5" x2="15" y2="8.5" width="0.3048" layer="16"/>
+<wire x1="15" y1="10" x2="15" y2="8.5" width="0.3048" layer="16"/>
 <wire x1="15" y1="8.5" x2="15.5" y2="8" width="0.3048" layer="16"/>
 <wire x1="15.5" y1="8" x2="21" y2="8" width="0.3048" layer="16"/>
@@
 <wire x1="22" y1="7" x2="23.04" y2="7" width="0.3048" layer="1"/>
 <wire x1="23.04" y1="7" x2="23.31" y2="6.73" width="0.3048" layer="1"/>
+<wire x1="15" y1="10" x2="14.5" y2="10.5" width="0.3048" layer="16"/>
+<wire x1="14.5" y1="10.5" x2="11.5" y2="10.5" width="0.3048" layer="16"/>
+<wire x1="11.5" y1="10.5" x2="9.5" y2="12.5" width="0.3048" layer="16"/>
 </signal>
 <signal name="MOSI">
 <contactref element="CON1" pad="10"/>
 <contactref element="ISP" pad="4"/>
-<wire x1="11.19" y1="13.25" x2="11.19" y2="12.81" width="0.3048" layer="16"/>
-<wire x1="11.19" y1="12.81" x2="11.5" y2="12.5" width="0.3048" layer="16"/>
-<wire x1="11.5" y1="12.5" x2="15" y2="12.5" width="0.3048" layer="16"/>
+<wire x1="12.138" y1="12.5" x2="15" y2="12.5" width="0.3048" layer="16"/>
 <wire x1="15" y1="12.5" x2="15.5" y2="12" width="0.3048" layer="16"/>
 <wire x1="15.5" y1="12" x2="15.5" y2="10" width="0.3048" layer="16"/>
@@
 <wire x1="16" y1="9.5" x2="18" y2="9.5" width="0.3048" layer="1"/>
 <wire x1="18" y1="9.5" x2="18.23" y2="9.27" width="0.3048" layer="1"/>
+<wire x1="12.138" y1="12.5" x2="11.388" y2="13.25" width="0.3048" layer="16"/>
+<wire x1="11.19" y1="13.25" x2="11.388" y2="13.25" width="0.3048" layer="16"/>
 </signal>
 <signal name="+5V">

Commit message: Updated adapter to hirose mini usb connector
Parts:
- removed USB: (no value), con-usb-3:USB-MIC-S
- added X1: MINI-USB-UX60SC-MB-5ST, con-hirose:UX60SC-MB-5ST
Connections:
- net GND: now also X1.5; no longer USB.GND, USB.P$11, USB.P$12, USB.P$13, USB.P$14
- net N$9: now also X1.1; no longer USB.VBUS
- net USBDM: now also X1.2; no longer USB.D-
- net USBDP: now also X1.3; no longer USB.D+
Routing:
- net N$9: track 23.2 -> 20.2 mm
- net USBDM: track 10.6 -> 10.1 mm
Other:
- board text added: "FH Kiel mrShark Adapter v0.0.3a"
- board text removed: "FH Kiel mrShark Adapter v0.0.1a"
Changed lines of the file:
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@@
 <text x="8.5" y="21" size="0.6096" layer="25" font="vector" ratio="15">FH Kiel
 mrShark Adapter
-v0.0.1a</text>
+v0.0.3a</text>
 <wire x1="24" y1="13.5" x2="17.5" y2="13.5" width="0.3048" layer="51"/>
 <wire x1="17.5" y1="13.5" x2="17.5" y2="5" width="0.3048" layer="51"/>
@@
 <attribute name="VALUE" x="2.246" y="8.619" size="0.0254" layer="27"/>
 </element>
-<element name="USB" library="con-usb-3" package="USB-MIC-S" value="" x="15" y="30.5" smashed="yes" rot="R180">
-<attribute name="NAME" x="18.81" y="25.23" size="0.6096" layer="25" rot="R180"/>
-</element>
 <element name="D1" library="diode" package="SOD323-R" value="PMEG2010EA" x="14" y="7" smashed="yes" rot="R270">
 <attribute name="NAME" x="15.5" y="5.9" size="0.6096" layer="25" rot="R90"/>
@@
 <attribute name="NAME" x="19.3838" y="3.8288" size="1.016" layer="25" ratio="10"/>
 <attribute name="VALUE" x="25.215" y="5.46" size="1.27" layer="27" rot="R90"/>
+</element>
+<element name="X1" library="con-hirose" package="UX60SC-MB-5ST" value="MINI-USB-UX60SC-MB-5ST" x="14.986" y="30.48" smashed="yes" rot="R270">
+<attribute name="NAME" x="19.558" y="29.17" size="0.6096" layer="25"/>
+<attribute name="VALUE" x="8.001" y="28.575" size="1.27" layer="27" rot="R270"/>
 </element>
 </elements>
@@
 <contactref element="IC4" pad="20"/>
 <contactref element="TP3" pad="TP"/>
-<contactref element="USB" pad="P$11"/>
-<contactref element="USB" pad="P$13"/>
-<contactref element="USB" pad="P$12"/>
-<contactref element="USB" pad="GND"/>
-<contactref element="USB" pad="P$14"/>
 <contactref element="ISP" pad="6"/>
 <polygon width="0.3048" layer="1" spacing="0.254" isolate="0.3048">
@@
 <via x="8.5" y="17.5" extent="1-16" drill="0.3048" shape="octagon"/>
 <via x="9" y="2.5" extent="1-16" drill="0.3048" shape="octagon"/>
+<contactref element="X1" pad="5"/>
 </signal>
 <signal name="INT1">
@@
 <signal name="USBDP">
 <contactref element="IC4" pad="14"/>
-<contactref element="USB" pad="D+"/>
-<wire x1="22.25" y1="22.3" x2="22.25" y2="23.25" width="0.3048" layer="16"/>
-<wire x1="22.25" y1="23.25" x2="22" y2="23.5" width="0.3048" layer="16"/>
-<wire x1="22" y1="23.5" x2="15.5" y2="23.5" width="0.3048" layer="16"/>
-<wire x1="15.5" y1="23.5" x2="15" y2="24" width="0.3048" layer="16"/>
-<via x="15" y="24" extent="1-16" drill="0.3048" shape="octagon"/>
-<wire x1="15" y1="24" x2="15" y2="26.2" width="0.3048" layer="1"/>
+<contactref element="X1" pad="3"/>
+<wire x1="22.25" y1="22.3" x2="22.25" y2="23.216" width="0.3048" layer="16"/>
+<wire x1="22.25" y1="23.216" x2="22.098" y2="23.368" width="0.3048" layer="16"/>
+<wire x1="22.098" y1="23.368" x2="18.796" y2="23.368" width="0.3048" layer="16"/>
+<via x="14.986" y="23.114" extent="1-16" drill="0.3048" shape="octagon"/>
+<wire x1="14.986" y1="23.114" x2="14.986" y2="24.38" width="0.3048" layer="1"/>
+<wire x1="18.796" y1="23.368" x2="17.526" y2="22.098" width="0.3048" layer="16"/>
+<wire x1="17.526" y1="22.098" x2="15.24" y2="22.098" width="0.3048" layer="16"/>
+<wire x1="15.24" y1="22.098" x2="14.986" y2="22.352" width="0.3048" layer="16"/>
+<wire x1="14.986" y1="22.352" x2="14.986" y2="23.114" width="0.3048" layer="16"/>
 </signal>
 <signal name="USBDM">
 <contactref element="IC4" pad="15"/>
-<contactref element="USB" pad="D-"/>
-<wire x1="15.65" y1="26.2" x2="15.65" y2="24.85" width="0.3048" layer="1"/>
-<wire x1="15.65" y1="24.85" x2="16" y2="24.5" width="0.3048" layer="1"/>
-<wire x1="16" y1="24.5" x2="16.5" y2="24.5" width="0.3048" layer="1"/>
-<via x="16.5" y="24.5" extent="1-16" drill="0.3048" shape="octagon"/>
-<wire x1="16.5" y1="24.5" x2="22.5" y2="24.5" width="0.3048" layer="16"/>
-<wire x1="22.75" y1="22.3" x2="22.75" y2="24.25" width="0.3048" layer="16"/>
-<wire x1="22.75" y1="24.25" x2="22.5" y2="24.5" width="0.3048" layer="16"/>
+<contactref element="X1" pad="2"/>
+<wire x1="22.75" y1="22.3" x2="22.75" y2="23.732" width="0.3048" layer="16"/>
+<wire x1="22.75" y1="23.732" x2="22.352" y2="24.13" width="0.3048" layer="16"/>
+<wire x1="22.352" y1="24.13" x2="18.288" y2="24.13" width="0.3048" layer="16"/>
+<wire x1="18.288" y1="24.13" x2="17.272" y2="23.114" width="0.3048" layer="16"/>
+<wire x1="17.272" y1="23.114" x2="16.51" y2="23.114" width="0.3048" layer="16"/>
+<wire x1="15.786" y1="24.38" x2="15.786" y2="23.33" width="0.3048" layer="1"/>
+<wire x1="15.786" y1="23.33" x2="16.002" y2="23.114" width="0.3048" layer="1"/>
+<via x="16.002" y="23.114" extent="1-16" drill="0.3048" shape="octagon"/>
+<wire x1="16.002" y1="23.114" x2="16.51" y2="23.114" width="0.3048" layer="16"/>
 </signal>
 <signal name="N$9">
-<contactref element="USB" pad="VBUS"/>
 <contactref element="D2" pad="A"/>
-<wire x1="16.3" y1="26.2" x2="16.8" y2="26.2" width="0.3048" layer="1"/>
-<wire x1="16.8" y1="26.2" x2="17.5" y2="25.5" width="0.3048" layer="1"/>
-<wire x1="17.5" y1="25.5" x2="17.5" y2="20.5" width="0.3048" layer="1"/>
-<wire x1="9" y1="19.5" x2="9" y2="18.5" width="0.3048" layer="1"/>
 <wire x1="9" y1="18.5" x2="9.5" y2="18" width="0.3048" layer="1"/>
 <wire x1="9.5" y1="18" x2="12" y2="18" width="0.3048" layer="1"/>
 <wire x1="12" y1="18" x2="12.5" y2="17.5" width="0.3048" layer="1"/>
 <wire x1="12.5" y1="17.5" x2="12.5" y2="14.6" width="0.3048" layer="1"/>
-<wire x1="9" y1="19.5" x2="9.5" y2="20" width="0.3048" layer="1"/>
-<wire x1="9.5" y1="20" x2="17" y2="20" width="0.3048" layer="1"/>
-<wire x1="17" y1="20" x2="17.5" y2="20.5" width="0.3048" layer="1"/>
+<contactref element="X1" pad="1"/>
+<wire x1="16.586" y1="24.38" x2="16.586" y2="23.8" width="0.3048" layer="1"/>
+<wire x1="16.586" y1="23.8" x2="17.018" y2="23.368" width="0.3048" layer="1"/>
+<wire x1="17.018" y1="23.368" x2="17.018" y2="20.574" width="0.3048" layer="1"/>
+<wire x1="17.018" y1="20.574" x2="16.51" y2="20.066" width="0.3048" layer="1"/>
+<wire x1="16.51" y1="20.066" x2="9.652" y2="20.066" width="0.3048" layer="1"/>
+<wire x1="9.652" y1="20.066" x2="9" y2="19.414" width="0.3048" layer="1"/>
+<wire x1="9" y1="18.5" x2="9" y2="19.414" width="0.3048" layer="1"/>
 </signal>
 <signal name="N$4">
